File: DSUB_KiCAD_Project.sch (KiCad schematic (older format))
At the start: 6 parts, among them J1 XT60-M, J2 XT60-M, J3 XT60-M, J4 XT60-M, J5 XT60-M, J6 Barrel_Jack

Commit message: Pcb made
actually made the pcb
Parts:
- removed J1, J2, J3, J4, J5: XT60-M, XT60-M:AMASS_XT60-M, symbol XT60-M:XT60-M
- removed J6: Barrel_Jack, Connector_BarrelJack:BarrelJack_CUI_PJ-036AH-SMT_Horizontal, symbol Connector:Barrel_Jack
Other:
- note removed: "Battery Pack Connectors"
- note removed: "Important: Should the Pack negative be directly connected to GND?\nThink this will Bypass the BMS system since everything else uses GND and not Pack-?\nMaybe we need separate the two grounds??\n-Seth"
- note removed: "Temperature Sensors"

Commit message: Changed layout
Layout was changed. Now we have planes for ground, 5v, and 3v3. hopefully current wont be an issue
Changed lines of the file:
@@
 F12 "Fire_redundant" I R 6750 5700 50
-$EndSheet
-$Sheet
-S 7400 4450 800  1400
-U 61B49F64
-F0 "sheet61B49F57" 50
-F1 "DSUB-plug.sch" 50
-F2 "t_mosi" I L 7400 4600 50
-F3 "t_miso" I L 7400 4750 50
-F4 "t_clk" I L 7400 4900 50
-F5 "Alert_scl" I L 7400 5050 50
-F6 "Alert_sda" I L 7400 5200 50
-F7 "Alert_Active" I L 7400 5350 50
-F8 "SWDIO" I L 7400 5500 50
-F9 "SWCLK" I L 7400 5650 50
-F10 "NRST" I R 8200 4600 50
-F11 "Fire" I R 8200 4750 50
-F12 "Fire_redundant" I R 8200 5750 50
 $EndSheet
 Text Label 5850 900  2    50   ~ 0
@@
 Text Label 5950 5600 2    50   ~ 0
 SWCLK
-Text Label 7400 4600 2    50   ~ 0
-tmosi
-Text Label 7400 4750 2    50   ~ 0
-tmiso
 Text Label 7400 4900 2    50   ~ 0
 t_clk
@@
 Text Label 6750 5700 0    50   ~ 0
 Fire_Redundant
+Text Label 8200 5750 0    50   ~ 0
+Fire_Redundant
+Text Label 8200 4750 0    50   ~ 0
+Fire
 Text Label 8200 4600 0    50   ~ 0
 NRT
-Text Label 8200 4750 0    50   ~ 0
-Fire
-Text Label 8200 5750 0    50   ~ 0
-Fire_Redundant
+Text Label 7400 4750 2    50   ~ 0
+tmiso
+Text Label 7400 4600 2    50   ~ 0
+tmosi
+$Sheet
+S 7400 4400 800  1400
+U 61AA7F18
+F0 "Sheet61AA7F17" 50
+F1 "DSUB-plug-power.sch" 50
+F2 "t_mosi" I L 7400 4600 50
+F3 "t_miso" I L 7400 4750 50
+F4 "t_clk" I L 7400 4900 50
+F5 "Alert_scl" I L 7400 5050 50
+F6 "Alert_sda" I L 7400 5200 50
+F7 "Alert_Active" I L 7400 5350 50
+F8 "SWDIO" I L 7400 5500 50
+F9 "SWCLK" I L 7400 5650 50
+F10 "NRST" I R 8200 4600 50
+F11 "Fire" I R 8200 4750 50
+F12 "Fire_redundant" I R 8200 5750 50
+$EndSheet
 $EndSCHEMATC
