File: Hardware/DSUB_KiCAD_Project.kicad_pcb (KiCad board)
At the start: 2 copper layers, 90.5 x 70 mm, 5 parts, among them J1 Telemetry Connector, J2 Data Connector, J3 Payload Connector, J4 Charges Connector, J6 Power Connector

Commit message: Added more silkscreen art
Parts:
- added G***: LOGO, Graphics:Orientation_Marker, B.Cu at (104.7, 90.0)
- added G***: LOGO, Graphics:RDT_Text, B.Cu at (122.3, 90.0)
Other:
- board text added: "DSUB Module Rev. 1"
- board text added: "THIS END TOWARDS TOP"
